Commit message: fix gripper urdf

File: Robots/robotiq/robotiq_2f_140_gripper_visualization/urdf/robotiq_arg2f.urdf (robot description, URDF)
Before this commit: robot robotiq_2f140, 3 links, 2 joints
Links:
- added link left_inner_finger, mass 0.0104003125914103; collision mesh filename=package://robotiq_2f_140_gripper_visualization/meshes/colli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; visual mesh filename=package://robotiq_2f_140_gripper_visualization/meshes/visua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
- added link left_inner_finger_pad; collision box size=0.03 0.07 0.0075; visual box size=0.027 0.065 0.0075
- added link left_inner_knuckle, mass 0.0271177346495152; collision mesh filename=package://robotiq_2f_140_gripper_visualization/meshes/colli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; visual mesh filename=package://robotiq_2f_140_gripper_visualization/meshes/visua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
- added link left_outer_finger, mass 0.022614240507152; collision mesh filename=package://robotiq_2f_140_gripper_visualization/meshes/colli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; visual mesh filename=package://robotiq_2f_140_gripper_visualization/meshes/visua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
- added link right_inner_finger, mass 0.0104003125914103; collision mesh filename=package://robotiq_2f_140_gripper_visualization/meshes/colli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; visual mesh filename=package://robotiq_2f_140_gripper_visualization/meshes/visua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
- added link right_inner_finger_pad; collision box size=0.03 0.07 0.0075; visual box size=0.027 0.065 0.0075
- added link right_inner_knuckle, mass 0.0271177346495152; collision mesh filename=package://robotiq_2f_140_gripper_visualization/meshes/colli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; visual mesh filename=package://robotiq_2f_140_gripper_visualization/meshes/visua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
- added link right_outer_finger, mass 0.022614240507152; collision mesh filename=package://robotiq_2f_140_gripper_visualization/meshes/colli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; visual mesh filename=package://robotiq_2f_140_gripper_visualization/meshes/visua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
Joints:
- added joint left_inner_finger_joint: type revolute, parent left_outer_finger, child left_inner_finger, origin xyz=0 0.0817554015893473 -0.0282203446692936 rpy=-0.725 0 0, axis 1 0 0, limit lower=-0.8757 upper=0.8757 effort=1000 velocity=2.0, mimic joint=finger_joint multiplier=1 offset=0
- added joint left_inner_finger_pad_joint: type fixed, parent left_inner_finger, child left_inner_finger_pad, origin xyz=0 0.0457554015893473 -0.0272203446692936 rpy=0 0 0, axis 0 0 1
- added joint left_inner_knuckle_joint: type revolute, parent robotiq_arg2f_base_link, child left_inner_knuckle, origin xyz=0 -0.0127 0.06142 rpy=2.2957 0 0, axis 1 0 0, limit lower=-0.8757 upper=0.8757 effort=1000 velocity=2.0, mimic joint=${prefix}finger_joint multiplier=-1 offset=0
- added joint left_outer_finger_joint: type fixed, parent left_outer_knuckle, child left_outer_finger, origin xyz=0 0.01821998610742 0.0260018192872234 rpy=0 0 0, axis 1 0 0
- added joint right_inner_finger_joint: type revolute, parent right_outer_finger, child right_inner_finger, origin xyz=0 0.0817554015893473 -0.0282203446692936 rpy=-0.725 0 0, axis 1 0 0, limit lower=-0.8757 upper=0.8757 effort=1000 velocity=2.0, mimic joint=$finger_joint multiplier=1 offset=0
- added joint right_inner_finger_pad_joint: type fixed, parent right_inner_finger, child right_inner_finger_pad, origin xyz=0 0.0457554015893473 -0.0272203446692936 rpy=0 0 0, axis 0 0 1
- added joint right_inner_knuckle_joint: type revolute, parent robotiq_arg2f_base_link, child right_inner_knuckle, origin xyz=0 0.0127 0.06142 rpy=2.29579 0 -3.14159, axis 1 0 0, limit lower=-0.8757 upper=0.8757 effort=1000 velocity=2.0, mimic joint=finger_joint multiplier=-1 offset=0
- added joint right_outer_finger_joint: type fixed, parent right_outer_knuckle, child right_outer_finger, origin xyz=0 0.01821998610742 0.0260018192872234 rpy=0 0 0, axis 1 0 0
